File: Electronics/2S charger/balenceCharger.brd (EAGLE design)
At the start: 100 x 80 mm, 24 parts, among them IC1 LM358N, J1 DCJ0202, Q1 BSS110, Q2 BSS110, Q3 BSS110, T1 2N2222

Commit message: error correction
Connections:
- removed net N$2: Q1.1, R1.2
- net N$1: now also R2.1
- net N$3: now also Q1.1, R1.2; no longer R2.1
Changed lines of the file:
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@@
 <wire x1="33.02" y1="19.05" x2="30.48" y2="19.05" width="0" layer="19" extent="1-1"/>
-</signal>
-<signal name="N$1">
-<contactref element="Q1" pad="2"/>
-<contactref element="T1" pad="3"/>
-<wire x1="10.16" y1="22.86" x2="6.35" y2="29.845" width="0" layer="19" extent="1-1"/>
-</signal>
-<signal name="N$2">
-<contactref element="R1" pad="2"/>
-<contactref element="Q1" pad="1"/>
-<wire x1="7.62" y1="27.94" x2="10.16" y2="27.94" width="0" layer="19" extent="1-1"/>
-</signal>
-<signal name="N$3">
-<contactref element="T1" pad="2"/>
-<contactref element="R2" pad="1"/>
-<wire x1="8.89" y1="20.32" x2="12.7" y2="22.86" width="0" layer="19" extent="1-1"/>
 </signal>
 <signal name="VCC">
@@
 <wire x1="17.78" y1="57.15" x2="27.69" y2="57.15" width="0" layer="19" extent="1-1"/>
 </signal>
+<signal name="N$1">
+<contactref element="T1" pad="3"/>
+<contactref element="R2" pad="1"/>
+<contactref element="Q1" pad="2"/>
+<wire x1="8.89" y1="20.32" x2="10.16" y2="22.86" width="0" layer="19" extent="1-1"/>
+<wire x1="6.35" y1="29.845" x2="10.16" y2="22.86" width="0" layer="19" extent="1-1"/>
+</signal>
+<signal name="N$3">
+<contactref element="R1" pad="2"/>
+<contactref element="Q1" pad="1"/>
+<contactref element="T1" pad="2"/>
+<wire x1="7.62" y1="27.94" x2="10.16" y2="27.94" width="0" layer="19" extent="1-1"/>
+<wire x1="12.7" y1="22.86" x2="10.16" y2="27.94" width="0" layer="19" extent="1-1"/>
+</signal>
 </signals>
